Commit message: 구체 추가

File: ros_gz_example_description/models/manipulator/model.urdf (robot description, URDF)
Before this commit: robot manipulator, 3 links, 2 joints
Links:
- added link sphere_link; visual mesh filename=package://ros_gz_example_description/models/manipulator/mes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 scale=0.02 0.02 0.02
Joints:
- added joint world_to_sphere: type fixed, parent world, child sphere_link, origin xyz=0.7 0 0 rpy=0 0 0

Commit message: ㅎㅎㅎ

File: ros_gz_example_description/models/manipulator/model.urdf (robot description, URDF)
Before this commit: robot manipulator, 4 links, 3 joints
Links:
- added link curvature_link; visual mesh filename=package://ros_gz_example_description/models/manipulator/mes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 scale=0.005 0.005 0.005
- link link_drone: geometry visual mesh filename=package://ros_gz_example_description/models/manipulator/mes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 scale=0.001 0.001 0.001
- link link_ee: geometry visual mesh filename=package://ros_gz_example_description/models/manipulator/mes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 scale=0.001 0.001 0.001
- link sphere_link: geometry visual mesh filename=package://ros_gz_example_description/models/manipulator/mes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 scale=0.006 0.006 0.006
Joints:
- added joint world_to_curvature: type fixed, parent world, child curvature_link, origin xyz=1.5 0.8 0 rpy=0 0 0
- joint world_to_sphere: origin xyz=0.7 0 0 rpy=0 0 0 -> xyz=1.5 -1.2 0 rpy=0 0 0

Commit message: 퇴근이다!

File: ros_gz_example_description/models/manipulator/model.urdf (robot description, URDF)
Before this commit: robot manipulator, 5 links, 4 joints
Links:
- link curvature_link: geometry visual mesh filename=package://ros_gz_example_description/models/manipulator/mes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 scale=0.004 0.004 0.004
